File: pcb/nano-supply-v1/nano-supply-v1.kicad_sch (KiCad schematic)
At the start: 49 parts, among them J1 USB_C_Receptacle_USB2.0_16P, J2 Conn_01x03_Pin, J3 IDC 2x8 SMD, J4 IDC 2x8 SMD, J5 IDC 2x8 SMD, J6 IDC 2x8 SMD, J7 IDC 2x8 SMD, J8 IDC 2x8 SMD, J9 Conn_01x02_Pin, Q1 AONR21307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

Commit message: routing
Changed lines of the file:
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@@
 	(wire
 		(pts
-			(xy 74.93 124.46) (xy 87.63 124.46)
+			(xy 243.84 33.02) (xy 264.16 33.02)
 		)
 		(stroke
@@
 	(wire
 		(pts
-			(xy 139.7 62.23) (xy 139.7 64.77)
+			(xy 74.93 124.46) (xy 87.63 124.46)
 		)
 		(stroke
@@
 	(wire
 		(pts
-			(xy 243.84 38.1) (xy 255.27 38.1)
+			(xy 139.7 62.23) (xy 139.7 64.77)
 		)
 		(stroke
@@
 	(wire
 		(pts
-			(xy 243.84 33.02) (xy 255.27 33.02)
-		)
-		(stroke
-			(width 0)
-			(type default)
-		)
-	)
-	(wire
-		(pts
 			(xy 91.44 116.84) (xy 104.14 116.84)
 		)
@@
 	(wire
 		(pts
+			(xy 243.84 38.1) (xy 264.16 38.1)
+		)
+		(stroke
+			(width 0)
+			(type default)
+		)
+	)
+	(wire
+		(pts
 			(xy 58.42 119.38) (xy 71.12 119.38)
 		)
@@
 	(wire
 		(pts
-			(xy 58.42 124.46) (xy 71.12 124.46)
+			(xy 243.84 43.18) (xy 264.16 43.18)
 		)
 		(stroke
@@
 	(wire
 		(pts
-			(xy 107.95 116.84) (xy 120.65 116.84)
+			(xy 58.42 124.46) (xy 71.12 124.46)
 		)
 		(stroke
@@
 	(wire
 		(pts
-			(xy 243.84 43.18) (xy 255.27 43.18)
+			(xy 107.95 116.84) (xy 120.65 116.84)
 		)
 		(stroke
@@
 	)
 	(label "EURO_P12"
-		(at 255.27 33.02 180)
+		(at 264.16 33.02 180)
 		(effects
 			(font
@@
 	)
 	(label "EURO_GND"
-		(at 255.27 38.1 180)
+		(at 264.16 38.1 180)
 		(effects
 			(font
@@
 	)
 	(label "EURO_N12"
-		(at 255.27 43.18 180)
+		(at 264.16 43.18 180)
 		(effects
 			(font
@@
 		(length 2.54)
 		(shape round)
-		(at 255.27 43.18 0)
+		(at 257.81 66.04 0)
 		(fields_autoplaced yes)
 		(effects
@@
 			(justify left bottom)
 		)
-		(property "Netclass" "POWER"
-			(at 255.9685 40.64 0)
+		(property "Netclass" "HIGH_POWER"
+			(at 258.5085 63.5 0)
+			(effects
+				(font
+					(size 1.27 1.27)
+				)
+				(justify left)
+			)
+		)
+		(property "Component Class" ""
+			(at 162.56 33.02 0)
+			(effects
+				(font
+					(size 1.27 1.27)
+					(italic yes)
+				)
+			)
+		)
+	)
+	(netclass_flag ""
+		(length 2.54)
+		(shape round)
+		(at 250.19 43.18 0)
+		(fields_autoplaced yes)
+		(effects
+			(font
+				(size 1.27 1.27)
+			)
+			(justify left bottom)
+		)
+		(property "Netclass" "HIGH_POWER"
+			(at 250.8885 40.64 0)
+			(effects
+				(font
+					(size 1.27 1.27)
+				)
+				(justify left)
+			)
+		)
+		(property "Component Class" ""
+			(at 154.94 10.16 0)
+			(effects
+				(font
+					(size 1.27 1.27)
+					(italic yes)
+				)
+			)
+		)
+	)
+	(netclass_flag ""
+		(length 2.54)
+		(shape round)
+		(at 250.19 38.1 0)
+		(fields_autoplaced yes)
+		(effects
+			(font
+				(size 1.27 1.27)
+			)
+			(justify left bottom)
+		)
+		(property "Netclass" "HIGH_POWER"
+			(at 250.8885 35.56 0)
 			(effects
 				(font
@@
 		)
 		(property "Component Class" ""
-			(at 160.02 10.16 0)
+			(at 154.94 5.08 0)
 			(effects
 				(font
@@
 			(justify left bottom)
 		)
-		(property "Netclass" "POWER"
+		(property "Netclass" "HIGH_POWER"
 			(at 262.3185 66.04 0)
 			(effects
@@
 		(length 2.54)
 		(shape round)
-		(at 190.5 33.02 0)
+		(at 250.19 33.02 0)
 		(fields_autoplaced yes)
 		(effects
@@
 			(justify left bottom)
 		)
-		(property "Netclass" "POWER"
-			(at 191.1985 30.48 0)
+		(property "Netclass" "HIGH_POWER"
+			(at 250.8885 30.48 0)
 			(effects
 				(font
@@
 		)
 		(property "Component Class" ""
-			(at 95.25 0 0)
+			(at 154.94 0 0)
 			(effects
 				(font
@@
 		(length 2.54)
 		(shape round)
-		(at 255.27 33.02 0)
+		(at 190.5 33.02 0)
 		(fields_autoplaced yes)
 		(effects
@@
 			(justify left bottom)
 		)
-		(property "Netclass" "POWER"
-			(at 255.9685 30.48 0)
+		(property "Netclass" "HIGH_POWER"
+			(at 191.1985 30.48 0)
 			(effects
 				(font
@@
 		)
 		(property "Component Class" ""
-			(at 160.02 0 0)
+			(at 95.25 0 0)
 			(effects
 				(font
@@
 		(length 2.54)
 		(shape round)
-		(at 255.27 38.1 0)
+		(at 22.86 64.77 0)
 		(fields_autoplaced yes)
 		(effects
@@
 		)
 		(property "Netclass" "POWER"
-			(at 255.9685 35.56 0)
+			(at 23.5585 62.23 0)
 			(effects
 				(font
@@
 		)
 		(property "Component Class" ""
-			(at 160.02 5.08 0)
+			(at -72.39 31.75 0)
 			(effects
 				(font
@@
 					(unit 1)
 				)
+			)
+		)
+	)
+	(symbol
+		(lib_id "power:GND")
+		(at 22.86 64.77 0)
+		(unit 1)
+		(exclude_from_sim no)
+		(in_bom yes)
+		(on_board yes)
+		(dnp no)
+		(fields_autoplaced yes)
+		(property "Reference" "#PWR018"
+			(at 22.86 71.12 0)
+			(effects
+				(font
+					(size 1.27 1.27)
+				)
+				(hide yes)
+			)
+		)
+		(property "Value" "GND"
+			(at 22.86 69.85 0)
+			(effects
+				(font
+					(size 1.27 1.27)
+				)
+			)
+		)
+		(property "Footprint" ""
+			(at 22.86 64.77 0)
+			(effects
+				(font
+					(size 1.27 1.27)
+				)
+				(hide yes)
+			)
+		)
+		(property "Datasheet" ""
+			(at 22.86 64.77 0)
+			(effects
+				(font
+					(size 1.27 1.27)
+				)
+				(hide yes)
+			)
+		)
+		(property "Description" "Power symbol creates a global label with name \"GND\" , ground"
+			(at 22.86 64.77 0)
+			(effects
+				(font
+					(size 1.27 1.27)
+				)
+				(hide yes)
+			)
+		)
+		(pin "1"
+		)
+		(instances
+			(project "nano-supply-v1"
+				(path "/318c286a-23d6-4ea5-8e60-705f90176dbf"
+					(reference "#PWR018")
+					(unit 1)
+				)
