File: pcb/nano-supply-v1/nano-supply-v1.kicad_sch (KiCad schematic)
At the start: 49 parts, among them J1 USB_C_Receptacle_USB2.0_16P, J2 Conn_01x03_Pin, J3 IDC 2x8 SMD, J4 IDC 2x8 SMD, J5 IDC 2x8 SMD, J6 IDC 2x8 SMD, J7 IDC 2x8 SMD, J8 IDC 2x8 SMD, J9 Conn_01x02_Pin, Q1 AONR21307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

Commit message: bom, gerber updates
Parts:
- R1: LCSC C22775 -> C22859
Changed lines of the file:
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@@
 			)
 		)
-		(property "LCSC" "C22775"
+		(property "LCSC" "C22859"
 			(at 102.87 40.6399 0)
 			(effects
