File: pcb/nano-supply-v1/nano-supply-v1.kicad_pcb (KiCad board)
At the start: 2 copper layers, 162 x 40 mm, 49 parts, among them J1 USB_C_Receptacle_USB2.0_16P, J2 Conn_01x03_Pin, J3 IDC 2x8 SMD, J4 IDC 2x8 SMD, J5 IDC 2x8 SMD, J6 IDC 2x8 SMD, J7 IDC 2x8 SMD, J8 IDC 2x8 SMD, J9 Conn_01x02_Pin, Q1 AONR21307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

Commit message: routing
Parts:
- moved U1 2.00 mm to (81.0, 93.0)
- moved C2 1.68 mm to (76.4, 83.5), turned to 180 degrees
- moved C12 1.20 mm to (150.0, 85.2)
- moved C15 1.20 mm to (190.0, 85.2)
- moved C10 0.40 mm to (150.0, 89.6)
- moved C13 0.30 mm to (190.0, 89.7)
- moved C5 0.30 mm to (111.5, 89.7)
- turned R3 to 180 degrees
Routing:
- net /EURO_P12: track 0.00 -> 160.4 mm, vias 0 -> 2
- net /EURO_P5: track 0.00 -> 144.2 mm, vias 0 -> 2
- net /EURO_N12: track 0.00 -> 126.8 mm
- net /20V: track 0.00 -> 55.7 mm, vias 0 -> 2
- net VBUS: track 0.00 -> 37.5 mm, vias 0 -> 2
- net /SCL: track 0.00 -> 18.1 mm
- net GND: track 0.00 -> 15.4 mm
- net /SDA: track 0.00 -> 14.9 mm
- net /D+: track 0.00 -> 13.1 mm, vias 0 -> 2
- net /D-: track 0.00 -> 12.1 mm
- net Net-(Q1-Pad4): track 0.00 -> 12.0 mm
- net /CC1: track 0.00 -> 8.84 mm, vias 0 -> 2
- net Net-(U1-ISET): track 0.00 -> 8.11 mm
- net Net-(U1-VSET): track 0.00 -> 7.99 mm
- net /CC2: track 0.00 -> 6.41 mm
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- added copper zone on B.Cu, net /EURO_GND
- added copper zone on F.Cu, net /EURO_GND
- added copper zone on B.Cu, net GND
- added copper zone on F.Cu, net GND

Commit message: stitching vias, routing tweaks
Routing:
- net /EURO_P5: track 144.2 -> 147.8 mm
- net GND: vias 0 -> 122
- net /EURO_GND: vias 0 -> 124
Other:
- board text added: "-12V (RED)"

Commit message: add jlc mappings etc
Parts:
- R5: value 5k1 -> 5.1k
