File: pcb/nano-supply-v2b/nano-supply-v2b.kicad_pcb (KiCad board)
At the start: 2 copper layers, 162 x 40 mm, 49 parts, among them J1 USB_C_Receptacle_USB2.0_16P, J2 Conn_01x03_Pin, J3 IDC 2x8 SMD, J4 IDC 2x8 SMD, J5 IDC 2x8 SMD, J6 IDC 2x8 SMD, J7 IDC 2x8 SMD, J8 IDC 2x8 SMD, J9 Conn_01x02_Pin, Q1 AONR21307, U1 HUSB238_xxxDD

Commit message: basic v2b fixes (footprints etc)
Parts:
- J1: footprint Connector_USB:USB_C_Receptacle_HRO_TYPE-C-31-M-12 -> nano-supply:TYPE-C-31-M-12
- J2: footprint Connector_PinHeader_2.54mm:PinHeader_1x03_P2.54mm_Vertical -> nano-supply:TestPads_1x03_P2.54mm; moved to B.Cu
- J9: footprint Connector_PinHeader_2.54mm:PinHeader_1x02_P2.54mm_Vertical -> nano-supply:TestPads_1x02_P2.54mm; moved to B.Cu
- moved VR2 2.01 mm to (88.3, 76.3)
- moved J2 0.44 mm to (70.2, 103.2), turned to 0 degrees
- turned J9 to 180 degrees
Routing:
- net /EURO_P5: track 147.8 -> 149.9 mm
- net /20V: track 55.7 -> 53.7 mm
- net VBUS: track 37.5 -> 38.2 mm, vias 2 -> 3
- net /D-: track 12.1 -> 12.7 mm
- net /SDA: track 14.9 -> 14.5 mm, vias 0 -> 1
- net /SCL: track 18.1 -> 17.8 mm, vias 0 -> 1
- net GND: vias 122 -> 0
- net /EURO_GND: vias 124 -> 0
Other:
- board text added: "v2"
- board text removed: "v1"

Commit message: basic power fixes
Parts:
- C10, C11, C12, C13, C14, C15, C3, C4, C5, C6, C7, C8, C9: footprint Capacitor_SMD:C_0805_2012Metric -> Capacitor_SMD:C_1206_3216Metric
- C2: value 10u -> 4.7u; footprint Capacitor_SMD:C_0805_2012Metric -> Capacitor_SMD:C_1206_3216Metric
- H1, H2: value MountingHole_Pad -> MountingHole; footprint MountingHole:MountingHole_3.2mm_M3_Pad -> MountingHole:MountingHole_3.2mm_M3
- R9: value 22k -> 10k
- moved Q1 5.33 mm to (81.7, 84.6), turned to 90 degrees
- moved C2 2.02 mm to (78.3, 84.2), turned to 90 degrees
- moved C3 1.40 mm to (83.0, 73.6), turned to 180 degrees
- moved C4 0.90 mm to (83.0, 76.1), turned to 180 degrees
- moved C10 0.60 mm to (150.0, 90.2)
- moved C12 0.60 mm to (150.0, 84.6)
- moved C15 0.60 mm to (190.0, 84.6)
- moved C11 0.60 mm to (150.0, 97.4)
- moved C14 0.60 mm to (190.0, 97.4)
- moved C6 0.60 mm to (111.5, 97.4)
- moved C9 0.60 mm to (111.5, 84.6)
- moved C13 0.50 mm to (190.0, 90.2)
- moved C5 0.50 mm to (111.5, 90.2)
- moved C7 0.40 mm to (83.0, 78.6), turned to 180 degrees
- moved R5 0.30 mm to (82.7, 99.0)
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Routing:
- net /EURO_P12: track 160.4 -> 0.00 mm, vias 2 -> 0
- net /EURO_P5: track 149.9 -> 0.00 mm, vias 2 -> 0
- net /EURO_N12: track 126.8 -> 0.00 mm
- net /20V: track 53.7 -> 0.00 mm, vias 2 -> 0
- net VBUS: track 38.2 -> 0.00 mm, vias 3 -> 0
- net /SCL: track 17.8 -> 0.00 mm, vias 1 -> 0
- net GND: track 15.4 -> 0.00 mm
- net /SDA: track 14.5 -> 0.00 mm, vias 1 -> 0
- net /D+: track 13.1 -> 0.00 mm, vias 2 -> 0
- net /D-: track 12.7 -> 0.00 mm
- net Net-(Q1-Pad4): track 12.0 -> 0.00 mm
- net /CC1: track 8.84 -> 0.00 mm, vias 2 -> 0
- net Net-(U1-ISET): track 8.11 -> 0.00 mm
- net Net-(U1-VSET): track 7.99 -> 0.00 mm
- net /CC2: track 6.41 -> 0.00 mm
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
Commit message: basic board routing
Parts:
- added D5: BZT52C15, Diode_SMD:D_SOD-123, F.Cu at (82.6, 105.7)
- added Q2: MMBT3904, Package_TO_SOT_SMD:SOT-23, F.Cu at (72.5, 82.1)
- added R10: 47k, Resistor_SMD:R_0603_1608Metric, F.Cu at (75.1, 82.1)
- added R11: 3.3k, Resistor_SMD:R_0805_2012Metric, F.Cu at (70.9, 78.6)
- added U2: LTV-817S, Package_DIP:SMDIP-4_W9.53mm, F.Cu at (75.1, 98.9)
- D1: value LED -> XL-3210SURUGC; footprint LED_SMD:LED_Kingbright_APA1606_1.6x0.6mm_Horizontal -> nano-supply:XL-3210SURUGC
- R6: value 22k -> 1.5k; footprint Resistor_SMD:R_0603_1608Metric -> Resistor_SMD:R_0805_2012Metric
- moved R6 20.2 mm to (82.6, 101.1), turned to -90 degrees
- moved R5 6.20 mm to (82.9, 92.8), turned to 90 degrees
- moved R4 3.74 mm to (82.9, 95.9)
- moved U1 2.51 mm to (78.5, 93.1)
- moved C9 2.20 mm to (111.6, 82.4)
- moved D1 0.45 mm to (69.8, 82.1)
Connections:
- D1 pad 1: Net-(D1-K) -> Net-(D1-GA)
- D1 pad 2: /20V -> GND
- J3 pad 13: unconnected-(J3-Pin_13-Pad13) -> Net-(J3-Pin_13)
- J3 pad 14: unconnected-(J3-Pin_14-Pad14) -> Net-(J3-Pin_13)
- J3 pad 15: unconnected-(J3-Pin_15-Pad15) -> Net-(J3-Pin_15)
- J3 pad 16: unconnected-(J3-Pin_16-Pad16) -> Net-(J3-Pin_15)
- J4 pad 13: unconnected-(J4-Pin_13-Pad13) -> Net-(J3-Pin_13)
- J4 pad 14: unconnected-(J4-Pin_14-Pad14) -> Net-(J3-Pin_13)
- J4 pad 15: unconnected-(J4-Pin_15-Pad15) -> Net-(J3-Pin_15)
- J4 pad 16: unconnected-(J4-Pin_16-Pad16) -> Net-(J3-Pin_15)
- J5 pad 13: unconnected-(J5-Pin_13-Pad13) -> Net-(J3-Pin_13)
- J5 pad 14: unconnected-(J5-Pin_14-Pad14) -> Net-(J3-Pin_13)
- J5 pad 15: unconnected-(J5-Pin_15-Pad15) -> Net-(J3-Pin_15)
- J5 pad 16: unconnected-(J5-Pin_16-Pad16) -> Net-(J3-Pin_15)
- J6 pad 13: unconnected-(J6-Pin_13-Pad13) -> Net-(J3-Pin_13)
- J6 pad 14: unconnected-(J6-Pin_14-Pad14) -> Net-(J3-Pin_13)
- J6 pad 15: unconnected-(J6-Pin_15-Pad15) -> Net-(J3-Pin_15)
- J6 pad 16: unconnected-(J6-Pin_16-Pad16) -> Net-(J3-Pin_15)
- J7 pad 13: unconnected-(J7-Pin_13-Pad13) -> Net-(J3-Pin_13)
- J7 pad 14: unconnected-(J7-Pin_14-Pad14) -> Net-(J3-Pin_13)
- J7 pad 15: unconnected-(J7-Pin_15-Pad15) -> Net-(J3-Pin_15)
- J7 pad 16: unconnected-(J7-Pin_16-Pad16) -> Net-(J3-Pin_15)
- J8 pad 13: unconnected-(J8-Pin_13-Pad13) -> Net-(J3-Pin_13)
- J8 pad 14: unconnected-(J8-Pin_14-Pad14) -> Net-(J3-Pin_13)
- J8 pad 15: unconnected-(J8-Pin_15-Pad15) -> Net-(J3-Pin_15)
- J8 pad 16: unconnected-(J8-Pin_16-Pad16) -> Net-(J3-Pin_15)
- R6 pad 1: Net-(D1-K) -> Net-(R6-Pad1)
- R6 pad 2: GND -> Net-(D5-K)
Routing:
- net /EURO_P12: track 0.00 -> 172.9 mm, vias 0 -> 2
- net /EURO_N12: track 0.00 -> 152.5 mm
- net /EURO_P5: track 0.00 -> 150.2 mm, vias 0 -> 2
- net Net-(J3-Pin_15): track 0.00 -> 107.6 mm
- net Net-(J3-Pin_13): track 0.00 -> 101.4 mm
- net VBUS: track 0.00 -> 35.6 mm, vias 0 -> 1
- net /20V: track 0.00 -> 31.7 mm
- net Net-(Q2-B): track 0.00 -> 28.1 mm
- net /CC1: track 0.00 -> 19.5 mm, vias 0 -> 2
- net /D-: track 0.00 -> 19.1 mm, vias 0 -> 2
- net /CC2: track 0.00 -> 17.8 mm, vias 0 -> 2
- net /D+: track 0.00 -> 16.9 mm, vias 0 -> 3
- net /SCL: track 0.00 -> 15.7 mm, vias 0 -> 1
- net /SDA: track 0.00 -> 12.1 mm, vias 0 -> 1
- net GND: track 0.00 -> 9.99 mm, vias 0 -> 4
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Other:
- board text removed: "HUSB238"
