File: pcb/nano-supply-v2b/nano-supply-v2b.kicad_pcb (KiCad board)
At the start: 2 copper layers, 162 x 40 mm, 54 parts, among them J1 USB_C_Receptacle_USB2.0_16P, J2 Conn_01x03_Pin, J3 IDC 2x8 SMD, J4 IDC 2x8 SMD, J5 IDC 2x8 SMD, J6 IDC 2x8 SMD, J7 IDC 2x8 SMD, J8 IDC 2x8 SMD, J9 Conn_01x02_Pin, Q1 AONR21307, Q2 MMBT3904, U1 HUSB238_xxxDD, U2 LTV-817S

Commit message: board finish
Routing:
- net Net-(J3-Pin_13): track 101.4 -> 109.0 mm
- net GND: vias 4 -> 111
- net /EURO_GND: vias 0 -> 285
Other:
- board text removed: "OK"
