File: pcb/nano-supply-v2b/nano-supply-v2b.kicad_sch (KiCad schematic)
At the start: 49 parts, among them J1 USB_C_Receptacle_USB2.0_16P, J2 Conn_01x03_Pin, J3 IDC 2x8 SMD, J4 IDC 2x8 SMD, J5 IDC 2x8 SMD, J6 IDC 2x8 SMD, J7 IDC 2x8 SMD, J8 IDC 2x8 SMD, J9 Conn_01x02_Pin, Q1 AONR21307, U1 HUSB238_xxxDD

Commit message: basic v2b fixes (footprints etc)
Parts:
- J1: footprint Connector_USB:USB_C_Receptacle_HRO_TYPE-C-31-M-12 -> nano-supply:TYPE-C-31-M-12
- J2: footprint Connector_PinHeader_2.54mm:PinHeader_1x03_P2.54mm_Vertical -> nano-supply:TestPads_1x03_P2.54mm
- J9: footprint Connector_PinHeader_2.54mm:PinHeader_1x02_P2.54mm_Vertical -> nano-supply:TestPads_1x02_P2.54mm
Connections:
- net GND: now also J1.SH (SHIELD); no longer J1.S1 (SHIELD)
Changed lines of the file:
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@@
 			)
 		)
-		(property "Footprint" "Connector_USB:USB_C_Receptacle_HRO_TYPE-C-31-M-12"
+		(property "Footprint" "nano-supply:TYPE-C-31-M-12"
 			(at 46.99 48.26 0)
 			(hide yes)
@@
 		(pin "B1"
 		)
-		(pin "S1"
+		(pin "SH"
 		)
 		(pin "A12"
@@
 			)
 		)
-		(property "Footprint" "Connector_PinHeader_2.54mm:PinHeader_1x02_P2.54mm_Vertical"
+		(property "Footprint" "nano-supply:TestPads_1x02_P2.54mm"
 			(at 67.31 85.09 0)
 			(hide yes)
@@
 			)
 		)
-		(property "Footprint" "Connector_PinHeader_2.54mm:PinHeader_1x03_P2.54mm_Vertical"
+		(property "Footprint" "nano-supply:TestPads_1x03_P2.54mm"
 			(at 152.4 64.77 0)
 			(hide yes)

Commit message: resistors, pdf
Parts:
- R9: value 22k -> 10k
Changed lines of the file:
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@@
 			)
 		)
-		(property "Value" "22k"
+		(property "Value" "10k"
 			(at 274.32 97.7899 0)
 			(show_name no)

Commit message: basic power fixes
Parts:
- removed H1, H2: MountingHole_Pad, MountingHole:MountingHole_3.2mm_M3_Pad, symbol Mechanical:MountingHole_Pad
- added H1, H2: MountingHole, MountingHole:MountingHole_3.2mm_M3, symbol Mechanical:MountingHole
- C10, C11, C12, C13, C14, C15, C3, C4, C5, C6, C7, C8, C9: footprint Capacitor_SMD:C_0805_2012Metric -> Capacitor_SMD:C_1206_3216Metric
- C2: value 10u -> 4.7u; footprint Capacitor_SMD:C_0805_2012Metric -> Capacitor_SMD:C_1206_3216Metric

Commit message: basic board routing
Parts:
- removed D1: LED, LED_SMD:LED_Kingbright_APA1606_1.6x0.6mm_Horizontal, symbol Device:LED
- added D1: XL-3210SURUGC, nano-supply:XL-3210SURUGC, symbol nano-supply:XL-3210SURUGC
- added D5: BZT52C15, Diode_SMD:D_SOD-123, symbol Device:D_Zener
- added Q2: MMBT3904, Package_TO_SOT_SMD:SOT-23, symbol Transistor_BJT:MMBT3904
- added R10: 47k, Resistor_SMD:R_0603_1608Metric, symbol Device:R
- added R11: 3.3k, Resistor_SMD:R_0805_2012Metric, symbol Device:R
- added U2: LTV-817S, Package_DIP:SMDIP-4_W9.53mm, symbol Isolator:LTV-817S
- R6: value 22k -> 1.5k; footprint Resistor_SMD:R_0603_1608Metric -> Resistor_SMD:R_0805_2012Metric; LCSC C31850 -> C23186
Connections:
- net EURO_N12: now also D5.2 (A)
- net EURO_P12: now also U2.1
- net GND: now also D1.2 (GK), Q2.2 (E), U2.3; no longer R6.2
- net VBUS: now also R10.1, R11.1
- net at J7.13 (Pin_13): now also J3.13 (Pin_13), J3.14 (Pin_14), J4.13 (Pin_13), J4.14 (Pin_14), J5.13 (Pin_13), J5.14 (Pin_14), J6.13 (Pin_13), J6.14 (Pin_14), J7.14 (Pin_14), J8.13 (Pin_13), J8.14 (Pin_14)
- net at J7.15 (Pin_15): now also J3.15 (Pin_15), J3.16 (Pin_16), J4.15 (Pin_15), J4.16 (Pin_16), J5.15 (Pin_15), J5.16 (Pin_16), J6.15 (Pin_15), J6.16 (Pin_16), J7.16 (Pin_16), J8.15 (Pin_15), J8.16 (Pin_16)
- net at R6.1: now also U2.2
- new net: D1.1 (GA), D1.3 (RA), R11.2
- new net: D1.4 (RK), Q2.3 (C)
- new net: D5.1 (K), R6.2
- new net: Q2.1 (B), R10.2, U2.4
Other:
- moved on the sheet: C10, C11, C12, C13, C14, C15, C5, C6, C9, H1, H2, H3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

Commit message: readme, license
Other:
- company: (none) -> github.com/xx0x/nano-supply
- title: (none) -> Nano Supply, USB-C PD PSU
Changed lines of the file:
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@@
 	(generator_version "10.0")
 	(paper "A4")
+	(title_block
+		(title "Nano Supply, USB-C PD PSU")
+		(date "2026-09-02")
+		(rev "v2b")
+		(company "github.com/xx0x/nano-supply")
+	)
 	(text "5k1 = approx 1.5A"
 		(exclude_from_sim no)
@@
 			(justify left bottom)
 		)
-		(property "Netclass" "HIGH_POWER"
+		(property "Net Class" "HIGH_POWER"
 			(at 250.8885 63.5 0)
 			(show_name no)
@@
 			(justify left bottom)
 		)
-		(property "Netclass" "HIGH_POWER"
+		(property "Net Class" "HIGH_POWER"
 			(at 250.8885 40.64 0)
 			(show_name no)
@@
 			(justify left bottom)
 		)
-		(property "Netclass" "HIGH_POWER"
+		(property "Net Class" "HIGH_POWER"
 			(at 250.8885 35.56 0)
 			(show_name no)
@@
 			(justify left bottom)
 		)
-		(property "Netclass" "HIGH_POWER"
+		(property "Net Class" "HIGH_POWER"
 			(at 254.6985 66.04 0)
 			(show_name no)
@@
 			(justify left bottom)
 		)
-		(property "Netclass" "HIGH_POWER"
+		(property "Net Class" "HIGH_POWER"
 			(at 250.8885 30.48 0)
 			(show_name no)
@@
 			(justify left bottom)
 		)
-		(property "Netclass" "HIGH_POWER"
+		(property "Net Class" "HIGH_POWER"
 			(at 191.1985 30.48 0)
 			(show_name no)
@@
 			(justify left bottom)
 		)
-		(property "Netclass" "POWER"
+		(property "Net Class" "POWER"
 			(at 23.5585 62.23 0)
 			(show_name no)
@@
 			(justify left bottom)
 		)
-		(property "Netclass" "POWER"
+		(property "Net Class" "POWER"
 			(at 68.0085 30.48 0)
 			(show_name no)

Commit message: add schematics notes
Other:
- note added: "Red LED has a lower forward voltage, will overtake green, making the circuit simpler."
- note added: "Requires at least 9V USB-PD, the LED will glow red on unsupported USB power supply."
Changed lines of the file:
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@@
 		(rev "v2b")
 		(company "github.com/xx0x/nano-supply")
+		(comment 1 "License: CERN-OHL-P-2.0")
 	)
 	(text "5k1 = approx 1.5A"
@@
 		(exclude_from_sim no)
 		(at 128.778 67.564 0)
+		(effects
+			(font
+				(size 1.27 1.27)
+			)
+		)
+	)
+	(text "Red LED has a lower forward voltage,\nwill overtake green, making the circuit simpler."
+		(exclude_from_sim no)
+		(at 197.358 97.536 0)
+		(effects
+			(font
+				(size 1.27 1.27)
+			)
+		)
+	)
+	(text "Requires at least 9V USB-PD, the LED will glow red on unsupported USB power supply."
+		(exclude_from_sim no)
+		(at 73.914 19.558 0)
 		(effects
 			(font
@@
 			(justify left bottom)
 		)
-		(property "Net Class" "HIGH_POWER"
+		(property "Netclass" "HIGH_POWER"
 			(at 250.8885 63.5 0)
 			(show_name no)
@@
 			(justify left bottom)
 		)
-		(property "Net Class" "HIGH_POWER"
+		(property "Netclass" "HIGH_POWER"
 			(at 250.8885 40.64 0)
 			(show_name no)
@@
 			(justify left bottom)
 		)
-		(property "Net Class" "HIGH_POWER"
+		(property "Netclass" "HIGH_POWER"
 			(at 250.8885 35.56 0)
 			(show_name no)
@@
 			(justify left bottom)
 		)
-		(property "Net Class" "HIGH_POWER"
+		(property "Netclass" "HIGH_POWER"
 			(at 254.6985 66.04 0)
 			(show_name no)
@@
 			(justify left bottom)
 		)
-		(property "Net Class" "HIGH_POWER"
+		(property "Netclass" "HIGH_POWER"
 			(at 250.8885 30.48 0)
 			(show_name no)
@@
 			(justify left bottom)
 		)
-		(property "Net Class" "HIGH_POWER"
+		(property "Netclass" "HIGH_POWER"
 			(at 191.1985 30.48 0)
 			(show_name no)
@@
 			(justify left bottom)
 		)
-		(property "Net Class" "POWER"
+		(property "Netclass" "POWER"
 			(at 23.5585 62.23 0)
 			(show_name no)
@@
 			(justify left bottom)
 		)
-		(property "Net Class" "POWER"
+		(property "Netclass" "POWER"
 			(at 68.0085 30.48 0)
 			(show_name no)
